Commit message: urdf 라이다 180도 변환 및 장애물 회피 튜닝추가

File: robot_controller/urdf/robot.urdf (robot description, URDF)
Before this commit: robot self_delivery_robot, 8 links, 7 joints
Joints:
- joint lidar_joint: origin xyz=0.160 0.0 0.355 rpy=0 0 3.14159 -> xyz=0.160 0.0 0.355 rpy=0 0 0

Commit message: urdf와 imu센서 ekf 완료 (현재 라이다 180도 뒤집힌 문제가 존재함)

File: robot_controller/urdf/robot.urdf (robot description, URDF)
Before this commit: robot self_delivery_robot, 8 links, 7 joints
Joints:
- joint imu_joint: origin xyz=0.160 0.0 0.325 rpy=0 0 0 -> xyz=0.180 0.0 0.6225 rpy=0 0 0
- joint lidar_joint: origin xyz=0.160 0.0 0.355 rpy=0 0 0 -> xyz=0.160 0.0 0.670 rpy=0 0 3.14159

Commit message: 피드포워드로 변경

File: robot_controller/urdf/robot.urdf (robot description, URDF)
Before this commit: robot self_delivery_robot, 8 links, 7 joints
Links:
- link base_link: mass 12.0 -> 10.0
- link wheel_front_left_link: geometry collision cylinder length=0.05 radius=0.06; visual cylinder length=0.05 radius=0.06
- link wheel_front_right_link: geometry collision cylinder length=0.05 radius=0.06; visual cylinder length=0.05 radius=0.06
- link wheel_rear_left_link: geometry collision cylinder length=0.05 radius=0.06; visual cylinder length=0.05 radius=0.06
- link wheel_rear_right_link: geometry collision cylinder length=0.05 radius=0.06; visual cylinder length=0.05 radius=0.06
Joints:
- joint imu_joint: origin xyz=0.180 0.0 0.6225 rpy=0 0 0 -> xyz=0.160 0.0 0.325 rpy=0 0 0
- joint lidar_joint: origin xyz=0.160 0.0 0.670 rpy=0 0 3.14159 -> xyz=0.160 0.0 0.355 rpy=0 0 3.14159
- joint wheel_front_left_joint: origin xyz=0.25 0.255 0.04 rpy=0 0 0 -> xyz=0.25 0.255 0.06 rpy=0 0 0
- joint wheel_front_right_joint: origin xyz=0.25 -0.255 0.04 rpy=0 0 0 -> xyz=0.25 -0.255 0.06 rpy=0 0 0
- joint wheel_rear_left_joint: origin xyz=-0.25 0.255 0.04 rpy=0 0 0 -> xyz=-0.25 0.255 0.06 rpy=0 0 0
- joint wheel_rear_right_joint: origin xyz=-0.25 -0.255 0.04 rpy=0 0 0 -> xyz=-0.25 -0.255 0.06 rpy=0 0 0

Commit message: $최종 자율 주행 완료$

File: robot_controller/urdf/robot.urdf (robot description, URDF)
Before this commit: robot self_delivery_robot, 8 links, 7 joints
Links:
- link wheel_front_left_link: geometry collision cylinder length=0.08 radius=0.06; visual cylinder length=0.08 radius=0.06
- link wheel_front_right_link: geometry collision cylinder length=0.08 radius=0.06; visual cylinder length=0.08 radius=0.06
- link wheel_rear_left_link: geometry collision cylinder length=0.08 radius=0.06; visual cylinder length=0.08 radius=0.06
- link wheel_rear_right_link: geometry collision cylinder length=0.08 radius=0.06; visual cylinder length=0.08 radius=0.06
Joints:
- joint imu_joint: origin xyz=0.160 0.0 0.325 rpy=0 0 0 -> xyz=0.18 0.0 0.6225 rpy=0 0 0
- joint lidar_joint: origin xyz=0.160 0.0 0.355 rpy=0 0 3.14159 -> xyz=0.16 0.0 0.67 rpy=0 0 3.14159
